Commit message: Unit changed as mm for HC10 and GP7

File: motoman_gp7_support/urdf/gp7_macro.xacro (robot description, xacro)
@@ -10,91 +10,56 @@
         <visual>
             <geometry>
-                <mesh filename="package://motoman_gp7_support/meshes/visual/gp7_base_link.stl"/>
+                <mesh filename="package://motoman_gp7_support/meshes/visual/gp7_base_link.stl" scale="1000 1000 1000" />
             </geometry>
             <material name="yaskawa_blue"/>
         </visual>
-        <collision>
-            <geometry>
-                <mesh filename="package://motoman_gp7_support/meshes/collision/gp7_base_link.stl"/>
-            </geometry>
-        </collision>
     </link>
     <link name="${prefix}link_1_s">
         <visual>
             <geometry>
-                <mesh filename="package://motoman_gp7_support/meshes/visual/gp7_link_1_s.stl"/>
+                <mesh filename="package://motoman_gp7_support/meshes/visual/gp7_link_1_s.stl" scale="1000 1000 1000" />
             </geometry>
             <material name="yaskawa_blue"/>
         </visual>
-        <collision>
-            <geometry>
-                <mesh filename="package://motoman_gp7_support/meshes/collision/gp7_link_1_s.stl"/>
-            </geometry>
-        </collision>
     </link>
     <link name="${prefix}link_2_l">
         <visual>
             <geometry>
-                <mesh filename="package://motoman_gp7_support/meshes/visual/gp7_link_2_l.stl"/>
+                <mesh filename="package://motoman_gp7_support/meshes/visual/gp7_link_2_l.stl" scale="1000 1000 1000" />
             </geometry>
             <material name="yaskawa_blue"/>
         </visual>
-        <collision>
-            <geometry>
-                <mesh filename="package://motoman_gp7_support/meshes/collision/gp7_link_2_l.stl"/>
-            </geometry>
-        </collision>
     </link>
     <link name="${prefix}link_3_u">
         <visual>
             <geometry>
-                <mesh filename="package://motoman_gp7_support/meshes/visual/gp7_link_3_u.stl"/>
+                <mesh filename="package://motoman_gp7_support/meshes/visual/gp7_link_3_u.stl" scale="1000 1000 1000" />
             </geometry>
             <material name="yaskawa_blue"/>
         </visual>
-        <collision>
-            <geometry>
-                <mesh filename="package://motoman_gp7_support/meshes/collision/gp7_link_3_u.stl"/>
-            </geometry>
-        </collision>
     </link>
     <link name="${prefix}link_4_r">
         <visual>
             <geometry>
-                <mesh filename="package://motoman_gp7_support/meshes/visual/gp7_link_4_r.stl"/>
+                <mesh filename="package://motoman_gp7_support/meshes/visual/gp7_link_4_r.stl" scale="1000 1000 1000" />
             </geometry>
             <material name="yaskawa_blue"/>
         </visual>
-        <collision>
-            <geometry>
-                <mesh filename="package://motoman_gp7_support/meshes/collision/gp7_link_4_r.stl"/>
-            </geometry>
-        </collision>
     </link>
     <link name="${prefix}link_5_b">
         <visual>
             <geometry>
-                <mesh filename="package://motoman_gp7_support/meshes/visual/gp7_link_5_b.stl"/>
+                <mesh filename="package://motoman_gp7_support/meshes/visual/gp7_link_5_b.stl" scale="1000 1000 1000" />
             </geometry>
             <material name="yaskawa_blue"/>
         </visual>
-        <collision>
-            <geometry>
-                <mesh filename="package://motoman_gp7_support/meshes/collision/gp7_link_5_b.stl"/>
-            </geometry>
-        </collision>
     </link>
     <link name="${prefix}link_6_t">
         <visual>
             <geometry>
-                <mesh filename="package://motoman_gp7_support/meshes/visual/gp7_link_6_t.stl"/>
+                <mesh filename="package://motoman_gp7_support/meshes/visual/gp7_link_6_t.stl" scale="1000 1000 1000" />
             </geometry>
             <material name="yaskawa_blue"/>
         </visual>
-        <collision>
-            <geometry>
-                <mesh filename="package://motoman_gp7_support/meshes/collision/gp7_link_6_t.stl"/>
-            </geometry>
-        </collision>
     </link>
     <link name="${prefix}tool0"/>
@@ -104,5 +69,5 @@
         <parent link="${prefix}base_link"/>
         <child link="${prefix}link_1_s"/>
-        <origin xyz="0 0 0.330" rpy="0 0 0" />
+        <origin xyz="0 0 330" rpy="0 0 0" />
         <axis xyz="0 0 1" />
         <limit lower="-2.9670" upper="2.9670" effort="212.66" velocity="6.5448"/>
@@ -111,5 +76,5 @@
         <parent link="${prefix}link_1_s"/>
         <child link="${prefix}link_2_l"/>
-        <origin xyz="0.040 0 0" rpy="0 0 0" />
+        <origin xyz="40 0 0" rpy="0 0 0" />
         <axis xyz="0 1 0" />
         <limit lower="-1.1344" upper="2.5307" effort="205.80" velocity="5.4977"/>
@@ -118,5 +83,5 @@
         <parent link="${prefix}link_2_l"/>
         <child link="${prefix}link_3_u"/>
-        <origin xyz="0 0 0.445" rpy="0 0 0" />
+        <origin xyz="0 0 445" rpy="0 0 0" />
         <axis xyz="0 -1 0" />
         <limit lower="-1.2217" upper="3.3161" effort="106.82" velocity="7.1558"/>
@@ -125,5 +90,5 @@
         <parent link="${prefix}link_3_u"/>
         <child link="${prefix}link_4_r"/>
-        <origin xyz="0.440 0 0.040" rpy="0 0 0" />
+        <origin xyz="440 0 40" rpy="0 0 0" />
         <axis xyz="-1 0 0" />
         <limit lower="-3.3161" upper="3.3161" effort="55.86" velocity="9.5993"/>
@@ -144,5 +109,5 @@
     </joint>
     <joint name="${prefix}joint_6_t-tool0" type="fixed">
-        <origin xyz="0.080 0 0" rpy="3.1415926 -1.570796 0"/>
+        <origin xyz="80 0 0" rpy="3.1415926 -1.570796 0"/>
         <parent link="${prefix}link_6_t"/>
         <child link="${prefix}tool0"/>
@@ -152,5 +117,5 @@
     <link name="${prefix}base" />
     <joint name="${prefix}base_link-base" type="fixed">
-        <origin xyz="0 0 0.330" rpy="0 0 0"/>
+        <origin xyz="0 0 330" rpy="0 0 0"/>
         <parent link="${prefix}base_link"/>
         <child link="${prefix}base"/>

File: motoman_hc10_support/urdf/hc10_macro.xacro (robot description, xacro)
@@ -10,5 +10,5 @@
       <visual>
         <geometry>
-          <mesh filename="package://motoman_hc10_support/meshes/hc10/visual/base_link.dae"/>
+          <mesh filename="package://motoman_hc10_support/meshes/hc10/visual/base_link.dae" scale="1000 1000 1000" />
         </geometry>
         <material name="yaskawa_blue"/>
@@ -16,5 +16,5 @@
       <collision>
         <geometry>
-          <mesh filename="package://motoman_hc10_support/meshes/hc10/collision/base_link.stl"/>
+          <mesh filename="package://motoman_hc10_support/meshes/hc10/collision/base_link.stl" scale="1000 1000 1000" />
         </geometry>
       </collision>
@@ -23,5 +23,5 @@
       <visual>
         <geometry>
-          <mesh filename="package://motoman_hc10_support/meshes/hc10/visual/link_1_s.dae"/>
+          <mesh filename="package://motoman_hc10_support/meshes/hc10/visual/link_1_s.dae" scale="1000 1000 1000" />
         </geometry>
         <material name="yaskawa_blue"/>
@@ -29,5 +29,5 @@
       <collision>
         <geometry>
-          <mesh filename="package://motoman_hc10_support/meshes/hc10/collision/link_1_s.stl"/>
+          <mesh filename="package://motoman_hc10_support/meshes/hc10/collision/link_1_s.stl" scale="1000 1000 1000" />
         </geometry>
       </collision>
@@ -36,5 +36,5 @@
       <visual>
         <geometry>
-          <mesh filename="package://motoman_hc10_support/meshes/hc10/visual/link_2_l.dae"/>
+          <mesh filename="package://motoman_hc10_support/meshes/hc10/visual/link_2_l.dae" scale="1000 1000 1000" />
         </geometry>
         <material name="yaskawa_blue"/>
@@ -42,5 +42,5 @@
       <collision>
         <geometry>
-          <mesh filename="package://motoman_hc10_support/meshes/hc10/collision/link_2_l.stl"/>
+          <mesh filename="package://motoman_hc10_support/meshes/hc10/collision/link_2_l.stl" scale="1000 1000 1000" />
         </geometry>
       </collision>
@@ -49,5 +49,5 @@
       <visual>
         <geometry>
-          <mesh filename="package://motoman_hc10_support/meshes/hc10/visual/link_3_u.dae"/>
+          <mesh filename="package://motoman_hc10_support/meshes/hc10/visual/link_3_u.dae" scale="1000 1000 1000" />
         </geometry>
         <material name="yaskawa_blue"/>
@@ -55,5 +55,5 @@
       <collision>
         <geometry>
-          <mesh filename="package://motoman_hc10_support/meshes/hc10/collision/link_3_u.stl"/>
+          <mesh filename="package://motoman_hc10_support/meshes/hc10/collision/link_3_u.stl" scale="1000 1000 1000" />
         </geometry>
       </collision>
@@ -62,5 +62,5 @@
       <visual>
         <geometry>
-          <mesh filename="package://motoman_hc10_support/meshes/hc10/visual/link_4_r.dae"/>
+          <mesh filename="package://motoman_hc10_support/meshes/hc10/visual/link_4_r.dae" scale="1000 1000 1000" />
         </geometry>
         <material name="yaskawa_blue"/>
@@ -68,5 +68,5 @@
       <collision>
         <geometry>
-          <mesh filename="package://motoman_hc10_support/meshes/hc10/collision/link_4_r.stl"/>
+          <mesh filename="package://motoman_hc10_support/meshes/hc10/collision/link_4_r.stl" scale="1000 1000 1000" />
         </geometry>
       </collision>
@@ -75,5 +75,5 @@
       <visual>
         <geometry>
-          <mesh filename="package://motoman_hc10_support/meshes/hc10/visual/link_5_b.dae"/>
+          <mesh filename="package://motoman_hc10_support/meshes/hc10/visual/link_5_b.dae" scale="1000 1000 1000" />
         </geometry>
         <material name="yaskawa_blue"/>
@@ -81,5 +81,5 @@
       <collision>
         <geometry>
-          <mesh filename="package://motoman_hc10_support/meshes/hc10/collision/link_5_b.stl"/>
+          <mesh filename="package://motoman_hc10_support/meshes/hc10/collision/link_5_b.stl" scale="1000 1000 1000" />
         </geometry>
       </collision>
@@ -88,5 +88,5 @@
       <visual>
         <geometry>
-          <mesh filename="package://motoman_hc10_support/meshes/hc10/visual/link_6_t.dae"/>
+          <mesh filename="package://motoman_hc10_support/meshes/hc10/visual/link_6_t.dae" scale="1000 1000 1000" />
         </geometry>
         <material name="yaskawa_blue"/>
@@ -94,5 +94,5 @@
       <collision>
         <geometry>
-          <mesh filename="package://motoman_hc10_support/meshes/hc10/collision/link_6_t.stl"/>
+          <mesh filename="package://motoman_hc10_support/meshes/hc10/collision/link_6_t.stl" scale="1000 1000 1000" />
         </geometry>
       </collision>
@@ -104,5 +104,5 @@
       <parent link="${prefix}base_link"/>
       <child link="${prefix}link_1_s"/>
-      <origin xyz="0 0 0.275" rpy="0 0 0" />
+      <origin xyz="0 0 275" rpy="0 0 0" />
       <axis xyz="0 0 1" />
       <limit lower="${radians(-180)}" upper="${radians(180)}" effort="368.48" velocity="${radians(130)}"/>
@@ -118,5 +118,5 @@
       <parent link="${prefix}link_2_l"/>
       <child link="${prefix}link_3_u"/>
-      <origin xyz="0 0 0.700" rpy="0 0 0" />
+      <origin xyz="0 0 700" rpy="0 0 0" />
       <axis xyz="0 -1 0" />
       <limit lower="${radians(-5)}" upper="${radians(355)}" effort="141.12" velocity="${radians(180)}"/>
@@ -125,5 +125,5 @@
       <parent link="${prefix}link_3_u"/>
       <child link="${prefix}link_4_r"/>
-      <origin xyz="0 0 -0.500" rpy="0 0 0" />
+      <origin xyz="0 0 -500" rpy="0 0 0" />
       <axis xyz="0 0 1" />
       <limit lower="${radians(-180)}" upper="${radians(180)}" effort="39.20" velocity="${radians(180)}"/>
@@ -132,5 +132,5 @@
       <parent link="${prefix}link_4_r"/>
       <child link="${prefix}link_5_b"/>
-      <origin xyz="0 0.162 0" rpy="0 0 0" />
+      <origin xyz="0 162 0" rpy="0 0 0" />
       <axis xyz="0 -1 0" />
       <limit lower="${radians(-180)}" upper="${radians(180)}" effort="31.36" velocity="${radians(250)}"/>
@@ -144,5 +144,5 @@
     </joint>
     <joint name="${prefix}joint_6_t-tool0" type="fixed">
-      <origin xyz="0 0 -0.130" rpy="${pi} 0 0"/>
+      <origin xyz="0 0 -130" rpy="${pi} 0 0"/>
       <parent link="${prefix}link_6_t"/>
       <child link="${prefix}tool0"/>
@@ -152,5 +152,5 @@
     <link name="${prefix}base" />
     <joint name="${prefix}base_link-base" type="fixed">
-      <origin xyz="0 0 0.275" rpy="0 0 0"/>
+      <origin xyz="0 0 275" rpy="0 0 0"/>
       <parent link="${prefix}base_link"/>
       <child link="${prefix}base"/>

File: motoman_hc10_support/urdf/hc10dt_macro.xacro (robot description, xacro)
@@ -13,5 +13,5 @@
       <visual>
         <geometry>
-          <mesh filename="package://motoman_hc10_support/meshes/hc10/visual/base_link.dae"/>
+          <mesh filename="package://motoman_hc10_support/meshes/hc10/visual/base_link.dae" scale="1000 1000 1000" />
         </geometry>
         <material name="yaskawa_blue"/>
@@ -19,5 +19,5 @@
       <collision>
         <geometry>
-          <mesh filename="package://motoman_hc10_support/meshes/hc10/collision/base_link.stl"/>
+          <mesh filename="package://motoman_hc10_support/meshes/hc10/collision/base_link.stl" scale="1000 1000 1000" />
         </geometry>
       </collision>
@@ -26,5 +26,5 @@
       <visual>
         <geometry>
-          <mesh filename="package://motoman_hc10_support/meshes/hc10/visual/link_1_s.dae"/>
+          <mesh filename="package://motoman_hc10_support/meshes/hc10/visual/link_1_s.dae" scale="1000 1000 1000" />
         </geometry>
         <material name="yaskawa_blue"/>
@@ -32,5 +32,5 @@
       <collision>
         <geometry>
-          <mesh filename="package://motoman_hc10_support/meshes/hc10/collision/link_1_s.stl"/>
+          <mesh filename="package://motoman_hc10_support/meshes/hc10/collision/link_1_s.stl" scale="1000 1000 1000" />
         </geometry>
       </collision>
@@ -39,5 +39,5 @@
       <visual>
         <geometry>
-          <mesh filename="package://motoman_hc10_support/meshes/hc10/visual/link_2_l.dae"/>
+          <mesh filename="package://motoman_hc10_support/meshes/hc10/visual/link_2_l.dae" scale="1000 1000 1000" />
         </geometry>
         <material name="yaskawa_blue"/>
@@ -45,5 +45,5 @@
       <collision>
         <geometry>
-          <mesh filename="package://motoman_hc10_support/meshes/hc10/collision/link_2_l.stl"/>
+          <mesh filename="package://motoman_hc10_support/meshes/hc10/collision/link_2_l.stl" scale="1000 1000 1000" />
         </geometry>
       </collision>
@@ -52,5 +52,5 @@
       <visual>
         <geometry>
-          <mesh filename="package://motoman_hc10_support/meshes/hc10/visual/link_3_u.dae"/>
+          <mesh filename="package://motoman_hc10_support/meshes/hc10/visual/link_3_u.dae" scale="1000 1000 1000" />
         </geometry>
         <material name="yaskawa_blue"/>
@@ -58,5 +58,5 @@
       <collision>
         <geometry>
-          <mesh filename="package://motoman_hc10_support/meshes/hc10/collision/link_3_u.stl"/>
+          <mesh filename="package://motoman_hc10_support/meshes/hc10/collision/link_3_u.stl" scale="1000 1000 1000" />
         </geometry>
       </collision>
@@ -65,5 +65,5 @@
       <visual>
         <geometry>
-          <mesh filename="package://motoman_hc10_support/meshes/hc10/visual/link_4_r.dae"/>
+          <mesh filename="package://motoman_hc10_support/meshes/hc10/visual/link_4_r.dae" scale="1000 1000 1000" />
         </geometry>
         <material name="yaskawa_blue"/>
@@ -71,5 +71,5 @@
       <collision>
         <geometry>
-          <mesh filename="package://motoman_hc10_support/meshes/hc10/collision/link_4_r.stl"/>
+          <mesh filename="package://motoman_hc10_support/meshes/hc10/collision/link_4_r.stl" scale="1000 1000 1000" />
         </geometry>
       </collision>
@@ -78,5 +78,5 @@
       <visual>
         <geometry>
-          <mesh filename="package://motoman_hc10_support/meshes/hc10/visual/link_5_b.dae"/>
+          <mesh filename="package://motoman_hc10_support/meshes/hc10/visual/link_5_b.dae" scale="1000 1000 1000" />
         </geometry>
         <material name="yaskawa_blue"/>
@@ -84,5 +84,5 @@
       <collision>
         <geometry>
-          <mesh filename="package://motoman_hc10_support/meshes/hc10/collision/link_5_b.stl"/>
+          <mesh filename="package://motoman_hc10_support/meshes/hc10/collision/link_5_b.stl" scale="1000 1000 1000" />
         </geometry>
       </collision>
@@ -91,5 +91,5 @@
       <visual>
         <geometry>
-          <mesh filename="package://motoman_hc10_support/meshes/hc10dt/visual/link_6_t.dae"/>
+          <mesh filename="package://motoman_hc10_support/meshes/hc10dt/visual/link_6_t.dae" scale="1000 1000 1000" />
         </geometry>
         <material name="yaskawa_blue"/>
@@ -97,5 +97,5 @@
       <collision>
         <geometry>
-          <mesh filename="package://motoman_hc10_support/meshes/hc10dt/collision/link_6_t.stl"/>
+          <mesh filename="package://motoman_hc10_support/meshes/hc10dt/collision/link_6_t.stl" scale="1000 1000 1000" />
        </geometry>
       </collision>
@@ -107,5 +107,5 @@
       <parent link="${prefix}base_link"/>
       <child link="${prefix}link_1_s"/>
-      <origin xyz="0 0 0.275" rpy="0 0 0" />
+      <origin xyz="0 0 275" rpy="0 0 0" />
       <axis xyz="0 0 1" />
       <limit lower="${radians(-180)}" upper="${radians(180)}" effort="368.48" velocity="${radians(130)}"/>
@@ -121,5 +121,5 @@
       <parent link="${prefix}link_2_l"/>
       <child link="${prefix}link_3_u"/>
-      <origin xyz="0 0 0.700" rpy="0 0 0" />
+      <origin xyz="0 0 700" rpy="0 0 0" />
       <axis xyz="0 -1 0" />
       <limit lower="${radians(-5)}" upper="${radians(355)}" effort="141.12" velocity="${radians(180)}"/>
@@ -128,5 +128,5 @@
       <parent link="${prefix}link_3_u"/>
       <child link="${prefix}link_4_r"/>
-      <origin xyz="0 0 -0.500" rpy="0 0 0" />
+      <origin xyz="0 0 -500" rpy="0 0 0" />
       <axis xyz="0 0 1" />
       <limit lower="${radians(-180)}" upper="${radians(180)}" effort="39.20" velocity="${radians(180)}"/>
@@ -135,5 +135,5 @@
       <parent link="${prefix}link_4_r"/>
       <child link="${prefix}link_5_b"/>
-      <origin xyz="0 0.162 0" rpy="0 0 0" />
+      <origin xyz="0 162 0" rpy="0 0 0" />
       <axis xyz="0 -1 0" />
       <limit lower="${radians(-180)}" upper="${radians(180)}" effort="31.36" velocity="${radians(250)}"/>
@@ -147,5 +147,5 @@
     </joint>
     <joint name="${prefix}joint_6_t-tool0" type="fixed">
-      <origin xyz="0 0 -0.170" rpy="${pi} 0 0"/>
+      <origin xyz="0 0 -170" rpy="${pi} 0 0"/>
       <parent link="${prefix}link_6_t"/>
       <child link="${prefix}tool0"/>
@@ -155,5 +155,5 @@
     <link name="${prefix}base" />
     <joint name="${prefix}base_link-base" type="fixed">
-      <origin xyz="0 0 0.275" rpy="0 0 0"/>
+      <origin xyz="0 0 275" rpy="0 0 0"/>
       <parent link="${prefix}base_link"/>
       <child link="${prefix}base"/>
